File: leds.sch (KiCad schematic (older format))
At the start: 55 parts, among them U1 TLC5955, U2 TLC5955, U3 TLC5955

Commit message: Updated for new KiCAD version (though still a few glitches in the schematics)
Parts:
- C20: footprint (none) -> w_smd_cap:c_elec_6.3x5.8
- LD1, LD10, LD11, LD12, LD13, LD14, LD15, LD16, LD17, LD18, LD19, LD2, LD20, LD21, LD22, LD23, LD24, LD25, LD26, LD27, LD28, LD29, LD3, LD30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: footprint (none) -> knielsenlib:RGB_0603
- U1, U2, U3: footprint (none) -> knielsenlib:TLC5955DCA
