File: leds.sch (KiCad schematic (older format))
At the start: 55 parts, among them U1 TLC5955, U2 TLC5955, U3 TLC5955

Commit message: Fix CSMALL <-> Csmall glitch when converting to new version
Parts:
- C1, C2, C3: symbol CSMALL -> Csmall
Changed lines of the file:
@@
 LIBS:w_opto
 LIBS:pcb_pov3d-cache
-EELAYER 24 0
+EELAYER 25 0
 EELAYER END
 $Descr A4 11693 8268
@@
 sout1
 $Comp
-L CSMALL C1
+L Csmall C1
 U 1 1 54AEF4F9
 P 9700 1400
@@
 $EndComp
 $Comp
-L CSMALL C2
+L Csmall C2
 U 1 1 54AEF50B
 P 9950 1400
@@
 $EndComp
 $Comp
-L CSMALL C3
+L Csmall C3
 U 1 1 54AEF51B
 P 10200 1400
