File: mcu_pwr.sch (KiCad schematic (older format))
At the start: 26 parts, among them P4 CONN_2, P5 KNUSB, U4 STM32F40X_LQFP64, U6 LP38691, X1 CRYSTAL

Commit message: Updated for new KiCAD version (though still a few glitches in the schematics)
Parts:
- B1: footprint (none) -> knielsenlib:SWITCH_FSMJSMA
- C14, C15: footprint (none) -> w_smd_cap:c_0805
- D1, D2: footprint (none) -> w_smd_leds:Led_0805
- JP1: footprint (none) -> w_pin_strip:pin_strip_3
- L1: footprint (none) -> SMD_Packages:SMD-0603
- P4: footprint (none) -> w_pin_strip:pin_strip_2-90
- P5: footprint (none) -> knielsenlib:10103594-0001LF
- R5, R6: footprint (none) -> w_smd_resistors:r_0805
- U4: footprint (none) -> knielsenlib:LQFP_64
- U6: footprint (none) -> knielsenlib:TO-252-3
- X1: footprint (none) -> knielsenlib:2-SOJ
Changed lines of the file:
@@
 LIBS:valves
 LIBS:w_opto
+LIBS:74xgxx
+LIBS:ac-dc
+LIBS:actel
+LIBS:brooktre
+LIBS:cmos_ieee
+LIBS:dc-dc
+LIBS:elec-unifil
+LIBS:ftdi
+LIBS:gennum
+LIBS:graphic
+LIBS:hc11
+LIBS:ir
+LIBS:logo
+LIBS:microchip_pic10mcu
+LIBS:microchip_pic12mcu
+LIBS:microchip_pic16mcu
+LIBS:microchip_pic18mcu
+LIBS:microchip_pic32mcu
+LIBS:motor_drivers
+LIBS:msp430
+LIBS:nordicsemi
+LIBS:nxp_armmcu
+LIBS:powerint
+LIBS:pspice
+LIBS:references
+LIBS:relays
+LIBS:rfcom
+LIBS:sensors
+LIBS:silabs
+LIBS:stm8
+LIBS:stm32
+LIBS:supertex
+LIBS:transf
+LIBS:ttl_ieee
+LIBS:video
 LIBS:pcb_pov3d-cache
-EELAYER 24 0
+EELAYER 25 0
 EELAYER END
 $Descr A4 11693 8268
@@
 F 0 "U4" H 2000 2450 60  0000 C CNN
 F 1 "STM32F40X_LQFP64" H 2050 1600 60  0000 C CNN
-F 2 "" H 2000 1150 60  0000 C CNN
+F 2 "knielsenlib:LQFP_64" H 2000 1150 60  0001 C CNN
 F 3 "" H 2000 1150 60  0000 C CNN
 	2    2000 2000
@@
 F 0 "B1" H 3407 1573 60  0000 C CNN
 F 1 "SWITCH_4PIN" H 3399 1095 60  0000 C CNN
-F 2 "" H 3400 1350 60  0001 C CNN
+F 2 "knielsenlib:SWITCH_FSMJSMA" H 3400 1350 60  0001 C CNN
 F 3 "" H 3400 1350 60  0001 C CNN
 	1    3400 1350
@@
 F 0 "X1" H 2850 2650 60  0000 C CNN
 F 1 "CRYSTAL" H 2850 2350 60  0000 C CNN
-F 2 "" H 2850 2500 60  0001 C CNN
+F 2 "knielsenlib:2-SOJ" H 2850 2500 60  0001 C CNN
 F 3 "" H 2850 2500 60  0001 C CNN
 	1    2850 2500
@@
 F 0 "U6" H 6050 1700 60  0000 C CNN
 F 1 "LP38691" H 6050 1350 60  0000 C CNN
-F 2 "" H 6050 1550 60  0001 C CNN
+F 2 "knielsenlib:TO-252-3" H 6050 1550 60  0001 C CNN
 F 3 "" H 6050 1550 60  0001 C CNN
 	1    6050 1550
@@
 F 0 "C15" H 6600 1900 50  0000 L CNN
 F 1 "2.2u" H 6600 1700 50  0000 L CNN
-F 2 "" H 6550 1800 60  0001 C CNN
+F 2 "w_smd_cap:c_0805" H 6550 1800 60  0001 C CNN
 F 3 "" H 6550 1800 60  0001 C CNN
 	1    6550 1800
@@
 F 0 "C14" H 5500 1900 50  0000 L CNN
 F 1 "2.2u" H 5500 1700 50  0000 L CNN
-F 2 "" H 5450 1800 60  0001 C CNN
+F 2 "w_smd_cap:c_0805" H 5450 1800 60  0001 C CNN
 F 3 "" H 5450 1800 60  0001 C CNN
 	1    5450 1800
@@
 F 0 "R6" V 5880 4550 50  0000 C CNN
 F 1 "1k" V 5800 4550 50  0000 C CNN
-F 2 "" H 5800 4550 60  0001 C CNN
+F 2 "w_smd_resistors:r_0805" H 5800 4550 60  0001 C CNN
 F 3 "" H 5800 4550 60  0001 C CNN
 	1    5800 4550
@@
 F 0 "R5" V 5880 4100 50  0000 C CNN
 F 1 "1k" V 5800 4100 50  0000 C CNN
-F 2 "" H 5800 4100 60  0001 C CNN
+F 2 "w_smd_resistors:r_0805" H 5800 4100 60  0001 C CNN
 F 3 "" H 5800 4100 60  0001 C CNN
 	1    5800 4100
@@
 F 0 "D2" H 6450 4650 50  0000 C CNN
 F 1 "SML-211YTT86" H 6450 4450 50  0000 C CNN
-F 2 "" H 6450 4550 60  0001 C CNN
+F 2 "w_smd_leds:Led_0805" H 6450 4550 60  0001 C CNN
 F 3 "" H 6450 4550 60  0001 C CNN
 	1    6450 4550
@@
 F 0 "D1" H 6450 4200 50  0000 C CNN
 F 1 "SML-211UTT86" H 6450 4000 50  0000 C CNN
-F 2 "" H 6450 4100 60  0001 C CNN
+F 2 "w_smd_leds:Led_0805" H 6450 4100 60  0001 C CNN
 F 3 "" H 6450 4100 60  0001 C CNN
 	1    6450 4100
@@
 F 0 "JP1" H 2700 4050 40  0000 L CNN
 F 1 "JUMPER3" H 2650 4250 40  0000 C CNN
-F 2 "" H 2650 4150 60  0001 C CNN
+F 2 "w_pin_strip:pin_strip_3" H 2650 4150 60  0001 C CNN
 F 3 "" H 2650 4150 60  0001 C CNN
 	1    2650 4150
@@
 F 0 "L1" V 2500 5350 40  0000 C CNN
 F 1 "30@100MHz" V 2650 5350 40  0000 C CNN
-F 2 "" H 2550 5350 60  0001 C CNN
+F 2 "SMD_Packages:SMD-0603" H 2550 5350 60  0001 C CNN
 F 3 "" H 2550 5350 60  0001 C CNN
 	1    2550 5350
@@
 F 0 "P5" H 2050 4450 60  0000 C CNN
 F 1 "KNUSB" H 2050 3750 60  0000 C CNN
-F 2 "" H 2050 4450 60  0001 C CNN
+F 2 "knielsenlib:10103594-0001LF" H 2050 4450 60  0001 C CNN
 F 3 "" H 2050 4450 60  0001 C CNN
 	1    2050 4450
@@
 F 0 "P4" V 1800 3950 40  0000 C CNN
 F 1 "CONN_2" V 1900 3950 40  0000 C CNN
-F 2 "" H 1850 3950 60  0000 C CNN
+F 2 "w_pin_strip:pin_strip_2-90" H 1850 3950 60  0001 C CNN
 F 3 "" H 1850 3950 60  0000 C CNN
 	1    1850 3950
