File: mcu_pwr.sch (KiCad schematic (older format))
At the start: 26 parts, among them P4 CONN_2, P5 KNUSB, U4 STM32F40X_LQFP64, U6 LP38691, X1 CRYSTAL

Commit message: Fix CSMALL <-> Csmall glitch when converting to new version
Parts:
- C10, C11, C12, C13, C16, C17, C18, C19, C6, C7, C8, C9: symbol CSMALL -> Csmall
Changed lines of the file:
@@
 LIBS:w_opto
 LIBS:pcb_pov3d-cache
-EELAYER 24 0
+EELAYER 25 0
 EELAYER END
 $Descr A4 11693 8268
@@
 	2400 1850 2500 1850
 $Comp
-L CSMALL C16
+L Csmall C16
 U 1 1 54A99019
 P 2600 1850
@@
 $EndComp
 $Comp
-L CSMALL C13
+L Csmall C13
 U 1 1 54A9901F
 P 2600 1700
@@
 $EndComp
 $Comp
-L CSMALL C17
+L Csmall C17
 U 1 1 54A9905B
 P 3100 2000
@@
 $EndComp
 $Comp
-L CSMALL C19
+L Csmall C19
 U 1 1 54A9906D
 P 3150 2800
@@
 $EndComp
 $Comp
-L CSMALL C18
+L Csmall C18
 U 1 1 54A99073
 P 3150 2200
@@
 	1450 1700 1450 1400
 $Comp
-L CSMALL C7
+L Csmall C7
 U 1 1 54A9911C
 P 1450 1300
@@
 $EndComp
 $Comp
-L CSMALL C8
+L Csmall C8
 U 1 1 54A9912E
 P 1650 1300
@@
 $EndComp
 $Comp
-L CSMALL C9
+L Csmall C9
 U 1 1 54A9913E
 P 1850 1300
@@
 Connection ~ 1650 1400
 $Comp
-L CSMALL C10
+L Csmall C10
 U 1 1 54A991B6
 P 2050 1300
@@
 $EndComp
 $Comp
-L CSMALL C11
+L Csmall C11
 U 1 1 54A991CA
 P 2250 1300
@@
 Connection ~ 2050 1400
 $Comp
-L CSMALL C12
+L Csmall C12
 U 1 1 54A99256
 P 2450 1300
@@
 $EndComp
 $Comp
-L CSMALL C6
+L Csmall C6
 U 1 1 54A99D22
 P 1250 1300
