File: pcb_pov3d.sch (KiCad schematic (older format))
At the start: 11 parts, among them P1 CONN_4X2, P2 CONN_6, P3 MICRO-SD, U4 STM32F40X_LQFP64, U5 US4881_HALL

Commit message: Misc. tweaks. Schematics is getting closer now.
Parts:
- added P6: CONN_12, symbol CONN_12
Connections:
- net labels added: pb0, pb1, pb12, pb2, pb8, pb9, usart3_rx, usart3_tx
- wire segments 100 -> 124
- no-connect marks 14 -> 6
Other:
- note added: "The sclk*, sin*, sout* and gsclk*\nare the high-speed signals. They\nshould be prioritised for optimal\nrouting."
- note removed: "?"
- moved on the sheet: R1, R2
Changed lines of the file:
@@
 Comment4 ""
 $EndDescr
-$Comp
-L STM32F40X_LQFP64 U4
-U 1 1 53591999
-P 2200 2200
-F 0 "U4" H 2200 3100 60  0000 C CNN
-F 1 "STM32F40X_LQFP64" H 2200 1300 60  0000 C CNN
-F 2 "" H 2200 1350 60  0000 C CNN
-F 3 "" H 2200 1350 60  0000 C CNN
-	1    2200 2200
-	1    0    0    -1
-$EndComp
 Text Label 7150 1450 0    60   ~ 0
 sin1
@@
 Text Notes 700  2550 0    30   ~ 0
 (bat_sense limited to\nPA0-7 / PB0-1 / PC0-5)
-Text Notes 3850 4000 0    120  ~ 24
+Text Notes 3900 4000 0    120  ~ 24
 Battery voltage monitoring
 $Comp
 L +5V #PWR06
 U 1 1 54AF57C6
-P 4200 4300
-F 0 "#PWR06" H 4200 4390 20  0001 C CNN
-F 1 "+5V" H 4200 4390 30  0000 C CNN
-F 2 "" H 4200 4300 60  0000 C CNN
-F 3 "" H 4200 4300 60  0000 C CNN
-	1    4200 4300
+P 4250 4300
+F 0 "#PWR06" H 4250 4390 20  0001 C CNN
+F 1 "+5V" H 4250 4390 30  0000 C CNN
+F 2 "" H 4250 4300 60  0000 C CNN
+F 3 "" H 4250 4300 60  0000 C CNN
+	1    4250 4300
 	1    0    0    -1
 $EndComp
@@
 L R R1
 U 1 1 54AF57F8
-P 4550 4400
-F 0 "R1" V 4630 4400 40  0000 C CNN
-F 1 "22k" V 4557 4401 40  0000 C CNN
-F 2 "" V 4480 4400 30  0000 C CNN
-F 3 "" H 4550 4400 30  0000 C CNN
-	1    4550 4400
+P 4600 4400
+F 0 "R1" V 4680 4400 40  0000 C CNN
+F 1 "22k" V 4607 4401 40  0000 C CNN
+F 2 "" V 4530 4400 30  0000 C CNN
+F 3 "" H 4600 4400 30  0000 C CNN
+	1    4600 4400
 	0    -1   -1   0
 $EndComp
@@
 L R R2
 U 1 1 54AF5864
-P 5450 4400
-F 0 "R2" V 5530 4400 40  0000 C CNN
-F 1 "10k" V 5457 4401 40  0000 C CNN
-F 2 "" V 5380 4400 30  0000 C CNN
-F 3 "" H 5450 4400 30  0000 C CNN
-	1    5450 4400
+P 5500 4400
+F 0 "R2" V 5580 4400 40  0000 C CNN
+F 1 "10k" V 5507 4401 40  0000 C CNN
+F 2 "" V 5430 4400 30  0000 C CNN
+F 3 "" H 5500 4400 30  0000 C CNN
+	1    5500 4400
 	0    -1   -1   0
 $EndComp
-Text Label 5000 4700 1    30   ~ 0
+Text Label 5050 4700 1    30   ~ 0
 bat_sense
 $Comp
 L GND #PWR07
 U 1 1 54AF5B3C
-P 5850 4500
-F 0 "#PWR07" H 5850 4500 30  0001 C CNN
-F 1 "GND" H 5850 4430 30  0001 C CNN
-F 2 "" H 5850 4500 60  0000 C CNN
-F 3 "" H 5850 4500 60  0000 C CNN
-	1    5850 4500
+P 5900 4500
+F 0 "#PWR07" H 5900 4500 30  0001 C CNN
+F 1 "GND" H 5900 4430 30  0001 C CNN
+F 2 "" H 5900 4500 60  0000 C CNN
+F 3 "" H 5900 4500 60  0000 C CNN
+	1    5900 4500
 	1    0    0    -1
 $EndComp
@@
 Text Notes 5800 5750 0    120  ~ 24
 GPIO
-Text Notes 5800 6750 0    360  ~ 72
-?
 $Comp
 L US4881_HALL U5
@@
 	1    0    0    -1
 $EndComp
-Text Label 4150 6450 0    60   ~ 12
+Text Label 4150 6450 0    60   ~ 0
 hall
 $Comp
@@
 	1    0    0    -1
 $EndComp
-NoConn ~ 2650 1400
-NoConn ~ 2650 1450
-NoConn ~ 2650 1500
-NoConn ~ 2650 1850
-NoConn ~ 2650 1800
-NoConn ~ 2650 1900
-NoConn ~ 2650 1950
-NoConn ~ 2650 2000
 NoConn ~ 1700 2900
 NoConn ~ 1700 2950
@@
 	7450 2050 7100 2050
 Wire Wire Line
-	5850 4400 5850 4500
-Wire Wire Line
-	5700 4400 5850 4400
-Connection ~ 5000 4400
-Wire Wire Line
-	5000 4400 5000 4750
-Wire Wire Line
-	4800 4400 5200 4400
-Wire Wire Line
-	4200 4400 4300 4400
-Wire Wire Line
-	4200 4300 4200 4400
+	5900 4400 5900 4500
+Wire Wire Line
+	5750 4400 5900 4400
+Connection ~ 5050 4400
+Wire Wire Line
+	5050 4400 5050 4750
+Wire Wire Line
+	4850 4400 5250 4400
+Wire Wire Line
+	4250 4400 4350 4400
+Wire Wire Line
+	4250 4300 4250 4400
 Wire Wire Line
 	1700 2250 1450 2250
@@
 Wire Notes Line
 	650  830  2650 830
+Wire Wire Line
+	2650 1900 2900 1900
+Wire Wire Line
+	2900 1950 2650 1950
+Wire Wire Line
+	2900 2000 2650 2000
+Text Label 2700 1900 0    30   ~ 0
+usart3_tx
+Text Label 2700 1950 0    30   ~ 0
+usart3_rx
+Text Label 2700 2000 0    30   ~ 0
+pb12
+$Comp
+L STM32F40X_LQFP64 U4
+U 1 1 53591999
+P 2200 2200
+F 0 "U4" H 2200 3100 60  0000 C CNN
+F 1 "STM32F40X_LQFP64" H 2200 1300 60  0000 C CNN
+F 2 "" H 2200 1350 60  0000 C CNN
+F 3 "" H 2200 1350 60  0000 C CNN
+	1    2200 2200
+	1    0    0    -1
+$EndComp
+Wire Wire Line
+	2650 1850 2900 1850
+Wire Wire Line
+	2900 1800 2650 1800
+Text Label 2700 1800 0    30   ~ 0
+pb8
+Text Label 2700 1850 0    30   ~ 0
+pb9
+Wire Wire Line
+	2650 1400 2900 1400
+Wire Wire Line
+	2900 1450 2650 1450
+Wire Wire Line
+	2650 1500 2900 1500
+Text Label 2700 1400 0    30   ~ 0
+pb0
+Text Label 2700 1450 0    30   ~ 0
+pb1
+Text Label 2700 1500 0    30   ~ 0
+pb2
+$Comp
+L CONN_12 P6
+U 1 1 54B2C91E
+P 6300 6550
+F 0 "P6" V 6250 6550 60  0000 C CNN
+F 1 "CONN_12" V 6350 6550 60  0000 C CNN
+F 2 "" H 6300 6550 60  0000 C CNN
+F 3 "" H 6300 6550 60  0000 C CNN
+	1    6300 6550
+	1    0    0    -1
+$EndComp
+Wire Wire Line
+	5450 6000 5950 6000
+Wire Wire Line
+	5600 6200 5950 6200
+Wire Wire Line
+	5600 6300 5950 6300
+Wire Wire Line
+	5950 6400 5600 6400
+Wire Wire Line
+	5600 6500 5950 6500
+Wire Wire Line
+	5600 6600 5950 6600
+Wire Wire Line
+	5600 6700 5950 6700
+Wire Wire Line
+	5950 6800 5600 6800
+Wire Wire Line
+	5600 6900 5950 6900
+Wire Wire Line
+	5450 7000 5950 7000
+Wire Wire Line
+	5450 7100 5950 7100
+Text Label 5650 6200 0    60   ~ 0
+pb0
+Text Label 5650 6300 0    60   ~ 0
+pb1
+Text Label 5650 6400 0    60   ~ 0
+pb2
+Text Label 5650 6500 0    60   ~ 0
+pb8
+Text Label 5650 6600 0    60   ~ 0
+pb9
+Text Label 5650 6700 0    60   ~ 0
+pb12
+Text Label 5600 6800 0    60   ~ 0
+usart3_tx
+Text Label 5600 6900 0    60   ~ 0
+usart3_rx
+Wire Wire Line
+	5450 6000 5450 6050
+$Comp
+L GND #PWR012
+U 1 1 54B2D861
+P 5450 6050
+F 0 "#PWR012" H 5450 6050 30  0001 C CNN
+F 1 "GND" H 5450 5980 30  0001 C CNN
+F 2 "" H 5450 6050 60  0000 C CNN
+F 3 "" H 5450 6050 60  0000 C CNN
+	1    5450 6050
+	1    0    0    -1
+$EndComp
+Wire Wire Line
+	5450 7100 5450 7150
+$Comp
+L GND #PWR013
+U 1 1 54B2D97E
+P 5450 7150
+F 0 "#PWR013" H 5450 7150 30  0001 C CNN
+F 1 "GND" H 5450 7080 30  0001 C CNN
+F 2 "" H 5450 7150 60  0000 C CNN
+F 3 "" H 5450 7150 60  0000 C CNN
+	1    5450 7150
+	1    0    0    -1
+$EndComp
+Wire Wire Line
+	5450 7000 5450 6950
+$Comp
+L +3.3V #PWR014
+U 1 1 54B2DA9C
+P 5450 6950
+F 0 "#PWR014" H 5450 6910 30  0001 C CNN
+F 1 "+3.3V" H 5450 7060 30  0000 C CNN
+F 2 "" H 5450 6950 60  0000 C CNN
+F 3 "" H 5450 6950 60  0000 C CNN
+	1    5450 6950
+	1    0    0    -1
+$EndComp
+$Comp
+L +3.3V #PWR015
+U 1 1 54B2DAED
+P 5500 6150
+F 0 "#PWR015" H 5500 6110 30  0001 C CNN
+F 1 "+3.3V" H 5500 6260 30  0000 C CNN
+F 2 "" H 5500 6150 60  0000 C CNN
+F 3 "" H 5500 6150 60  0000 C CNN
+	1    5500 6150
+	-1   0    0    1
+$EndComp
+Wire Wire Line
+	5500 6150 5500 6100
+Wire Wire Line
+	5500 6100 5950 6100
+Text Notes 2650 2600 0    40   ~ 0
+The sclk*, sin*, sout* and gsclk*\nare the high-speed signals. They\nshould be prioritised for optimal\nrouting.
+Wire Notes Line
+	2600 2500 3700 2500
+Wire Notes Line
+	3700 2500 3700 2800
+Wire Notes Line
+	3700 2800 2600 2800
+Wire Notes Line
+	2600 2800 2600 2500
 $EndSCHEMATC

Commit message: Tweaks.
Other:
- note added: "The pb* generic\nGPIOs could be\nswapped for some\nof the pc* if that\nsimplifies routing"
- moved on the sheet: P3, P6, R4, U5

Commit message: Updated for new KiCAD version (though still a few glitches in the schematics)
Parts:
- P1: footprint (none) -> w_pin_strip:pin_socket_4x2
- P2: footprint (none) -> w_pin_strip:pin_strip_6
- P3: footprint (none) -> knielsenlib:SD_502774
- P6: footprint (none) -> w_pin_strip:pin_strip_12-90
- R1, R2, R3, R4: footprint (none) -> w_smd_resistors:r_0805
- U4: footprint (none) -> knielsenlib:LQFP_64
- U5: footprint (none) -> Discret:TO92
Changed lines of the file:
@@
 LIBS:valves
 LIBS:w_opto
+LIBS:74xgxx
+LIBS:ac-dc
+LIBS:actel
+LIBS:brooktre
+LIBS:cmos_ieee
+LIBS:dc-dc
+LIBS:elec-unifil
+LIBS:ftdi
+LIBS:gennum
+LIBS:graphic
+LIBS:hc11
+LIBS:ir
+LIBS:logo
+LIBS:microchip_pic10mcu
+LIBS:microchip_pic12mcu
+LIBS:microchip_pic16mcu
+LIBS:microchip_pic18mcu
+LIBS:microchip_pic32mcu
+LIBS:motor_drivers
+LIBS:msp430
+LIBS:nordicsemi
+LIBS:nxp_armmcu
+LIBS:powerint
+LIBS:pspice
+LIBS:references
+LIBS:relays
+LIBS:rfcom
+LIBS:sensors
+LIBS:silabs
+LIBS:stm8
+LIBS:stm32
+LIBS:supertex
+LIBS:transf
+LIBS:ttl_ieee
+LIBS:video
 LIBS:pcb_pov3d-cache
-EELAYER 24 0
+EELAYER 25 0
 EELAYER END
 $Descr A4 11693 8268
@@
 F 0 "P1" H 2300 4600 50  0000 C CNN
 F 1 "CONN_4X2" V 2300 4350 40  0000 C CNN
-F 2 "" H 2300 4350 60  0000 C CNN
+F 2 "w_pin_strip:pin_socket_4x2" H 2300 4350 60  0001 C CNN
 F 3 "" H 2300 4350 60  0000 C CNN
 	1    2300 4350
@@
 F 0 "R3" V 3380 4650 40  0000 C CNN
 F 1 "47k" V 3307 4651 40  0000 C CNN
-F 2 "" V 3230 4650 30  0000 C CNN
+F 2 "w_smd_resistors:r_0805" V 3230 4650 30  0001 C CNN
 F 3 "" H 3300 4650 30  0000 C CNN
 	1    3300 4650
@@
 F 0 "P3" H 1900 5800 60  0000 C CNN
 F 1 "MICRO-SD" H 1900 7000 60  0000 C CNN
-F 2 "" H 1900 6400 60  0001 C CNN
+F 2 "knielsenlib:SD_502774" H 1900 6400 60  0001 C CNN
 F 3 "" H 1900 6400 60  0001 C CNN
 	1    1900 6400
@@
 F 0 "R4" V 3030 6000 40  0000 C CNN
 F 1 "47k" V 2957 6001 40  0000 C CNN
-F 2 "" V 2880 6000 30  0000 C CNN
+F 2 "w_smd_resistors:r_0805" V 2880 6000 30  0001 C CNN
 F 3 "" H 2950 6000 30  0000 C CNN
 	1    2950 6000
@@
 F 0 "R1" V 4680 4400 40  0000 C CNN
 F 1 "22k" V 4607 4401 40  0000 C CNN
-F 2 "" V 4530 4400 30  0000 C CNN
+F 2 "w_smd_resistors:r_0805" V 4530 4400 30  0001 C CNN
 F 3 "" H 4600 4400 30  0000 C CNN
 	1    4600 4400
@@
 F 0 "R2" V 5580 4400 40  0000 C CNN
 F 1 "10k" V 5507 4401 40  0000 C CNN
-F 2 "" V 5430 4400 30  0000 C CNN
+F 2 "w_smd_resistors:r_0805" V 5430 4400 30  0001 C CNN
 F 3 "" H 5500 4400 30  0000 C CNN
 	1    5500 4400
@@
 F 0 "P2" V 8250 4450 60  0000 C CNN
 F 1 "CONN_6" V 8350 4450 60  0000 C CNN
-F 2 "" H 8300 4450 60  0000 C CNN
+F 2 "w_pin_strip:pin_strip_6" H 8300 4450 60  0001 C CNN
 F 3 "" H 8300 4450 60  0000 C CNN
 	1    8300 4450
@@
 F 0 "U5" H 4650 5850 60  0000 C CNN
 F 1 "US4881_HALL" H 4650 6400 60  0000 C CNN
-F 2 "" H 4650 6200 60  0000 C CNN
+F 2 "Discret:TO92" H 4650 6200 60  0001 C CNN
 F 3 "" H 4650 6200 60  0000 C CNN
 	1    4650 6200
@@
 F 0 "U4" H 2200 3100 60  0000 C CNN
 F 1 "STM32F40X_LQFP64" H 2200 1300 60  0000 C CNN
-F 2 "" H 2200 1350 60  0000 C CNN
+F 2 "knielsenlib:LQFP_64" H 2200 1350 60  0001 C CNN
 F 3 "" H 2200 1350 60  0000 C CNN
 	1    2200 2200
@@
 F 0 "P6" V 6250 6450 60  0000 C CNN
 F 1 "CONN_12" V 6350 6450 60  0000 C CNN
-F 2 "" H 6300 6450 60  0000 C CNN
+F 2 "w_pin_strip:pin_strip_12-90" H 6300 6450 60  0001 C CNN
 F 3 "" H 6300 6450 60  0000 C CNN
 	1    6300 6450
