File: pcb_pov3d.sch (KiCad schematic (older format))
At the start: 12 parts, among them P1 CONN_4X2, P2 CONN_6, P3 MICRO-SD, P6 CONN_12, U4 STM32F40X_LQFP64, U5 US4881_HALL

Commit message: Fix CSMALL <-> Csmall glitch when converting to new version
Parts:
- C4, C5: symbol CSMALL -> Csmall
Changed lines of the file:
@@
 LIBS:w_opto
 LIBS:pcb_pov3d-cache
-EELAYER 24 0
+EELAYER 25 0
 EELAYER END
 $Descr A4 11693 8268
@@
 nrf_miso
 $Comp
-L CSMALL C5
+L Csmall C5
 U 1 1 54AE0171
 P 2800 6300
@@
 $EndComp
 $Comp
-L CSMALL C4
+L Csmall C4
 U 1 1 54B151E6
 P 4100 6150
