File: pcb_pov3d.kicad_pcb (KiCad board)
At the start: 4 copper layers, 98 x 90 mm, 95 parts, among them P1 CONN_4X2, P2 CONN_6, P3 MICRO-SD, P4 CONN_2, P5 KNUSB, P6 CONN_12, U1 TLC5955, U2 TLC5955, U3 TLC5955, U4 STM32F40X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

Commit message: Add pull-up and capacitor on Hall output
Parts:
- added C22: 4.7n, w_smd_cap:c_0805, B.Cu at (56.6, 117.3)
- added R7: 10k, w_smd_resistors:r_0805, B.Cu at (58.3, 119.1)
- D1: value Power -> SML-211UTT86
- D2: value User LED -> SML-211YTT86
- JP1: value BAT USB -> JUMPER3
- U4: value STM32F40X -> STM32F40X_LQFP64
Routing:
- net /hall: track 47.1 -> 53.1 mm
- net +3V3: track 170.3 -> 171.6 mm, vias 16 -> 17
- net GND: track 149.5 -> 150.8 mm, vias 79 -> 80
Changed lines of the file:
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@@
 (kicad_pcb (version 4) (host pcbnew "(after 2015-mar-04 BZR unknown)-product")
   (general
-    (links 347)
+    (links 351)
     (no_connects 0)
-    (area 50.949999 59.449999 149.050001 149.550001)
+    (area 50.949999 59.02092 149.050001 149.62946)
     (thickness 1.6)
     (drawings 50)
-    (tracks 2591)
+    (tracks 2602)
     (zones 0)
-    (modules 95)
+    (modules 97)
     (nets 208)
   )
@@
   )
   (setup
-    (last_trace_width 1.016)
+    (last_trace_width 0.2032)
     (user_trace_width 0.1524)
     (user_trace_width 0.2032)
@@
       (effects (font (size 1.09982 1.09982) (thickness 0.127)) (justify mirror))
     )
-    (fp_text value STM32F40X (at 0 -1.651 90) (layer B.SilkS)
+    (fp_text value STM32F40X_LQFP64 (at 0 -1.651 90) (layer B.SilkS)
       (effects (font (size 1.016 0.762) (thickness 0.1524)) (justify mirror))
     )
@@
       (effects (font (size 0.8001 0.8001) (thickness 0.14986)) (justify mirror))
     )
-    (fp_text value Power (at 0 -1.80086) (layer B.SilkS)
+    (fp_text value SML-211UTT86 (at 0 -1.80086) (layer B.SilkS)
       (effects (font (size 0.8001 0.8001) (thickness 0.14986)) (justify mirror))
     )
@@
       (effects (font (size 0.8001 0.8001) (thickness 0.14986)) (justify mirror))
     )
-    (fp_text value "User LED" (at 0 -1.80086) (layer B.SilkS)
+    (fp_text value SML-211YTT86 (at 0 -1.80086) (layer B.SilkS)
       (effects (font (size 1.016 0.8128) (thickness 0.14986)) (justify mirror))
     )
@@
       (effects (font (size 1.016 1.016) (thickness 0.2032)) (justify mirror))
     )
-    (fp_text value "BAT   USB" (at 0.1 3.6 180) (layer F.SilkS)
+    (fp_text value JUMPER3 (at 0.1 3.6 180) (layer F.SilkS)
       (effects (font (size 1.016 0.889) (thickness 0.2032)))
     )
@@
     (pad 1 thru_hole circle (at 0 0) (size 3.6 3.6) (drill 3.6) (layers *.Cu))
   )
+  (module w_smd_cap:c_0805 (layer B.Cu)
+    (at 56.6 117.3 45)
+    (descr "SMT capacitor, 0805")
+    (fp_text reference C22 (at 0 -1.555635 45) (layer B.SilkS)
+      (effects (font (size 1.016 0.8128) (thickness 0.1524)) (justify mirror))
+    )
+    (fp_text value 4.7n (at -2.474874 -0.494975 135) (layer B.SilkS)
+      (effects (font (size 1.016 0.8128) (thickness 0.1524)) (justify mirror))
+    )
+    (fp_line (start 0.635 0.635) (end 0.635 -0.635) (layer B.SilkS) (width 0.127))
+    (fp_line (start -0.635 0.635) (end -0.635 -0.6096) (layer B.SilkS) (width 0.127))
+    (fp_line (start -1.016 0.635) (end 1.016 0.635) (layer B.SilkS) (width 0.127))
+    (fp_line (start 1.016 0.635) (end 1.016 -0.635) (layer B.SilkS) (width 0.127))
+    (fp_line (start 1.016 -0.635) (end -1.016 -0.635) (layer B.SilkS) (width 0.127))
+    (fp_line (start -1.016 -0.635) (end -1.016 0.635) (layer B.SilkS) (width 0.127))
+    (pad 1 smd rect (at 0.9525 0 45) (size 1.30048 1.4986) (layers B.Cu B.Paste B.Mask)
+      (net 2 GND))
+    (pad 2 smd rect (at -0.9525 0 45) (size 1.30048 1.4986) (layers B.Cu B.Paste B.Mask)
+      (net 197 /hall))
+    (model walter\smd_cap\c_0805.wrl
+      (at (xyz 0 0 0))
+      (scale (xyz 1 1 1))
+      (rotate (xyz 0 0 0))
+    )
+  )
+  (module w_smd_resistors:r_0805 (layer B.Cu)
+    (at 58.3 119.1 45)
+    (descr "SMT resistor, 0805")
+    (fp_text reference R7 (at 0.070711 1.767767 45) (layer B.SilkS)
+      (effects (font (size 1.016 0.8128) (thickness 0.1524)) (justify mirror))
+    )
+    (fp_text value 10k (at 2.899138 0.212132 135) (layer B.SilkS)
+      (effects (font (size 1.016 0.8128) (thickness 0.1524)) (justify mirror))
+    )
+    (fp_line (start 0.635 0.635) (end 0.635 -0.635) (layer B.SilkS) (width 0.127))
+    (fp_line (start -0.635 0.635) (end -0.635 -0.6096) (layer B.SilkS) (width 0.127))
+    (fp_line (start -1.016 0.635) (end 1.016 0.635) (layer B.SilkS) (width 0.127))
+    (fp_line (start 1.016 0.635) (end 1.016 -0.635) (layer B.SilkS) (width 0.127))
+    (fp_line (start 1.016 -0.635) (end -1.016 -0.635) (layer B.SilkS) (width 0.127))
+    (fp_line (start -1.016 -0.635) (end -1.016 0.635) (layer B.SilkS) (width 0.127))
+    (pad 1 smd rect (at 0.9525 0 45) (size 1.30048 1.4986) (layers B.Cu B.Paste B.Mask)
+      (net 207 +3V3))
+    (pad 2 smd rect (at -0.9525 0 45) (size 1.30048 1.4986) (layers B.Cu B.Paste B.Mask)
+      (net 197 /hall))
+    (model walter/smd_resistors/r_0805.wrl
+      (at (xyz 0 0 0))
+      (scale (xyz 1 1 1))
+      (rotate (xyz 0 0 0))
+    )
+  )
   (gr_text VCC (at 70.8 95.4 90) (layer B.SilkS)
     (effects (font (size 1.27 1.27) (thickness 0.1778)) (justify mirror))
@@
   (segment (start 81.79526 100.9493) (end 82 101.15404) (width 0.2032) (layer B.Cu) (net 1))
   (segment (start 80.83006 100.9493) (end 81.79526 100.9493) (width 0.2032) (layer B.Cu) (net 1))
+  (segment (start 57.273519 116.626481) (end 57.973519 116.626481) (width 0.2032) (layer B.Cu) (net 2))
+  (segment (start 57.973519 116.626481) (end 58.4 116.2) (width 0.2032) (layer B.Cu) (net 2))
+  (via (at 58.4 116.2) (size 0.635) (layers F.Cu B.Cu) (net 2))
   (segment (start 80.445123 87.054877) (end 78.9 85.509754) (width 1.016) (layer B.Cu) (net 2))
   (via (at 78.9 85.5) (size 0.635) (layers F.Cu B.Cu) (net 2))
@@
   (segment (start 82.409612 101.590388) (end 83.522301 100.477699) (width 0.2032) (layer B.Cu) (net 196))
   (segment (start 81.79526 97.44918) (end 80.83006 97.44918) (width 0.2032) (layer B.Cu) (net 196))
+  (segment (start 57.626481 119.773519) (end 56.027775 121.372225) (width 0.2032) (layer B.Cu) (net 197))
+  (segment (start 56.027775 121.372225) (end 55.740956 121.372225) (width 0.2032) (layer B.Cu) (net 197))
+  (segment (start 55.926481 117.973519) (end 55.926481 121.1867) (width 0.2032) (layer B.Cu) (net 197))
+  (segment (start 55.926481 121.1867) (end 55.740956 121.372225) (width 0.2032) (layer B.Cu) (net 197))
   (segment (start 82.435116 93.959266) (end 84.222301 95.746451) (width 0.2032) (layer F.Cu) (net 197))
   (segment (start 71.87834 109.29641) (end 67.816771 109.29641) (width 0.2032) (layer F.Cu) (net 197))
@@
   (segment (start 76.550988 102.5) (end 78.050988 104) (width 0.2032) (layer F.Cu) (net 203))
   (segment (start 78.050988 104) (end 78.5 104) (width 0.2032) (layer F.Cu) (net 203))
+  (segment (start 60.1 118.219578) (end 60.1 118.1) (width 0.2032) (layer B.Cu) (net 207))
+  (segment (start 59.893097 118.426481) (end 60.1 118.219578) (width 0.2032) (layer B.Cu) (net 207))
+  (segment (start 58.973519 118.426481) (end 59.893097 118.426481) (width 0.2032) (layer B.Cu) (net 207))
+  (via (at 60.1 118.1) (size 0.635) (drill 0.3048) (layers F.Cu B.Cu) (net 207))
   (segment (start 69.486 84.014) (end 68.820408 84.679592) (width 1.016) (layer B.Cu) (net 207))
   (segment (start 69.486 83.82072) (end 69.486 84.014) (width 1.016) (layer B.Cu) (net 207))

Commit message: Misc. minor tweaks
Parts:
- D1: value SML-211UTT86 -> Power LED
- D2: value SML-211YTT86 -> User LED
- JP1: value JUMPER3 -> BAT USB
Changed lines of the file:
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@@
     (thickness 1.6)
     (drawings 50)
-    (tracks 2602)
+    (tracks 2601)
     (zones 0)
     (modules 97)
@@
       (effects (font (size 0.8001 0.8001) (thickness 0.14986)) (justify mirror))
     )
-    (fp_text value SML-211UTT86 (at 0 -1.80086) (layer B.SilkS)
+    (fp_text value "Power LED" (at 0 -1.80086) (layer B.SilkS)
       (effects (font (size 0.8001 0.8001) (thickness 0.14986)) (justify mirror))
     )
@@
       (effects (font (size 0.8001 0.8001) (thickness 0.14986)) (justify mirror))
     )
-    (fp_text value SML-211YTT86 (at 0 -1.80086) (layer B.SilkS)
+    (fp_text value "User LED" (at 0 -1.80086) (layer B.SilkS)
       (effects (font (size 1.016 0.8128) (thickness 0.14986)) (justify mirror))
     )
@@
       (effects (font (size 1.016 1.016) (thickness 0.2032)) (justify mirror))
     )
-    (fp_text value JUMPER3 (at 0.1 3.6 180) (layer F.SilkS)
+    (fp_text value "BAT   USB" (at 0.1 3.6 180) (layer F.SilkS)
       (effects (font (size 1.016 0.889) (thickness 0.2032)))
     )
@@
   (segment (start 82.922559 92.673519) (end 82.646059 92.673519) (width 0.2032) (layer B.Cu) (net 2))
   (segment (start 82.646059 92.673519) (end 81.726481 92.673519) (width 0.2032) (layer B.Cu) (net 2))
-  (segment (start 86.7 88.28) (end 86.43 88.01) (width 0.2032) (layer In2.Cu) (net 2))
   (segment (start 92.973519 92.026481) (end 93.373519 92.026481) (width 0.2032) (layer B.Cu) (net 2))
   (segment (start 87.7475 92.2) (end 86.8 92.2) (width 0.2032) (layer B.Cu) (net 2))
@@
   (segment (start 84.29914 126.80086) (end 84.4 126.7) (width 0.2032) (layer B.Cu) (net 171))
   (via (at 84.4 126.7) (size 0.635) (layers F.Cu B.Cu) (net 171))
-  (segment (start 93.97773 101.94752) (end 95.277699 100.647551) (width 0.2032) (layer B.Cu) (net 172))
-  (segment (start 95.277699 99.801295) (end 95.419044 99.65995) (width 0.2032) (layer B.Cu) (net 172))
   (segment (start 92.7325 101.94752) (end 93.97773 101.94752) (width 0.2032) (layer B.Cu) (net 172))
-  (segment (start 95.419044 99.65995) (end 96.376144 99.65995) (width 0.2032) (layer B.Cu) (net 172))
-  (segment (start 95.277699 100.647551) (end 95.277699 99.801295) (width 0.2032) (layer B.Cu) (net 172))
-  (segment (start 96.376144 99.65995) (end 96.825156 99.65995) (width 0.2032) (layer B.Cu) (net 172))
-  (segment (start 96.507657 99.342451) (end 96.825156 99.65995) (width 0.2032) (layer F.Cu) (net 172))
-  (segment (start 96.36883 81.87228) (end 96.36883 99.203624) (width 0.2032) (layer F.Cu) (net 172))
-  (segment (start 96.36883 99.203624) (end 96.507657 99.342451) (width 0.2032) (layer F.Cu) (net 172))
-  (segment (start 85.75024 71.25369) (end 96.36883 81.87228) (width 0.2032) (layer F.Cu) (net 172))
+  (segment (start 93.97773 101.94752) (end 95.277026 100.648224) (width 0.2032) (layer B.Cu) (net 172))
+  (segment (start 95.277026 100.648224) (end 95.277026 99.801968) (width 0.2032) (layer B.Cu) (net 172))
+  (segment (start 95.277026 99.801968) (end 95.418994 99.66) (width 0.2032) (layer B.Cu) (net 172))
+  (segment (start 95.418994 99.66) (end 96.45 99.66) (width 0.2032) (layer B.Cu) (net 172))
+  (segment (start 96.45 99.66) (end 96.57 99.78) (width 0.2032) (layer B.Cu) (net 172))
+  (segment (start 85.75024 71.25369) (end 96.322501 81.825951) (width 0.2032) (layer F.Cu) (net 172))
   (segment (start 85.75024 70.02448) (end 85.75024 71.25369) (width 0.2032) (layer F.Cu) (net 172))
-  (via (at 96.825156 99.65995) (size 0.635) (drill 0.3048) (layers F.Cu B.Cu) (net 172))
-  (segment (start 95.900019 99.833258) (end 95.900019 100.28227) (width 0.2032) (layer F.Cu) (net 173))
-  (segment (start 95.90641 99.826867) (end 95.900019 99.833258) (width 0.2032) (layer F.Cu) (net 173))
-  (segment (start 95.90641 81.98461) (end 95.90641 99.826867) (width 0.2032) (layer F.Cu) (net 173))
-  (segment (start 85.1 71.1782) (end 95.90641 81.98461) (width 0.2032) (layer F.Cu) (net 173))
+  (segment (start 96.322501 81.825951) (end 96.322501 99.083489) (width 0.2032) (layer F.Cu) (net 172))
+  (segment (start 96.57 99.330988) (end 96.57 99.78) (width 0.2032) (layer F.Cu) (net 172))
+  (segment (start 96.322501 99.083489) (end 96.57 99.330988) (width 0.2032) (layer F.Cu) (net 172))
+  (via (at 96.57 99.78) (size 0.635) (drill 0.3048) (layers F.Cu B.Cu) (net 172))
+  (segment (start 95.90641 99.826694) (end 95.899327 99.833777) (width 0.2032) (layer F.Cu) (net 173))
   (segment (start 85.1 70.02448) (end 85.1 71.1782) (width 0.2032) (layer F.Cu) (net 173))
+  (segment (start 95.90641 81.98461) (end 95.90641 99.826694) (width 0.2032) (layer F.Cu) (net 173))
+  (segment (start 94.0521 102.4479) (end 95.899327 100.600673) (width 0.2032) (layer B.Cu) (net 173))
+  (segment (start 95.899327 100.600673) (end 95.899327 100.282789) (width 0.2032) (layer B.Cu) (net 173))
+  (segment (start 95.899327 99.833777) (end 95.899327 100.282789) (width 0.2032) (layer F.Cu) (net 173))
+  (segment (start 85.1 71.1782) (end 95.90641 81.98461) (width 0.2032) (layer F.Cu) (net 173))
   (segment (start 92.7325 102.4479) (end 94.0521 102.4479) (width 0.2032) (layer B.Cu) (net 173))
-  (segment (start 94.0521 102.4479) (end 95.900019 100.599981) (width 0.2032) (layer B.Cu) (net 173))
-  (segment (start 95.900019 100.599981) (end 95.900019 100.28227) (width 0.2032) (layer B.Cu) (net 173))
-  (via (at 95.900019 100.28227) (size 0.635) (drill 0.3048) (layers F.Cu B.Cu) (net 173))
+  (via (at 95.899327 100.282789) (size 0.635) (drill 0.3048) (layers F.Cu B.Cu) (net 173))
   (segment (start 57.42782 94.8) (end 78.791745 94.8) (width 0.2032) (layer F.Cu) (net 174))
   (segment (start 78.791745 94.8) (end 79.936548 93.655197) (width 0.2032) (layer F.Cu) (net 174))

Commit message: Tweaks
Routing:
- net +5V: track 164.2 -> 163.6 mm
